Commit message: update

File: elfin_description/urdf/elfin_15F.urdf.xacro (robot description, xacro)
@@ -22,29 +22,29 @@
       link="elfin_base_link" />
     <child
-      link="elfin_base" />
-  </joint>
-  <link
-    name="elfin_base">
-    <inertial>
-      <origin
-        xyz="-0.00137018130408533 -2.08409607078014E-06 0.0376538014243397"
-        rpy="0 0 0" />
-      <mass
-        value="2.70257461902285" />
-      <inertia
-        ixx="0.00938125784352759"
-        ixy="-3.18876715466082E-09"
-        ixz="-6.88676148404872E-05"
-        iyy="0.00898645591278108"
-        iyz="-1.99352142230343E-07"
-        izz="0.015708544428067" />
-    </inertial>
-    <visual>
-      <origin
-        xyz="0 0 0"
-        rpy="0 0 0" />
-      <geometry>
-        <mesh
-          filename="package://elfin_description/meshes/elfin15_F/elfin_base.STL" />
+      link="base_link" />
+  </joint>
+  <link
+    name="base_link">
+    <inertial>
+      <origin
+        xyz="-0.000695002623445946 -5.07508519484099E-06 0.0375658828060339"
+        rpy="0 0 0" />
+      <mass
+        value="2.71888716466908" />
+      <inertia
+        ixx="0.00938317508875725"
+        ixy="-3.60387611495622E-08"
+        ixz="-6.88676148720587E-05"
+        iyy="0.00898832759881519"
+        iyz="-1.99352155737403E-07"
+        izz="0.0157105653615728" />
+    </inertial>
+    <visual>
+      <origin
+        xyz="0 0 0"
+        rpy="0 0 0" />
+      <geometry>
+        <mesh
+          filename="package://elfin_description/meshes/elfin15_F/base_link.STL" />
       </geometry>
       <material
@@ -60,5 +60,5 @@
       <geometry>
         <mesh
-          filename="package://elfin_description/meshes/elfin15_F/elfin_base.STL" />
+          filename="package://elfin_description/meshes/elfin15_F/base_link.STL" />
       </geometry>
     </collision>
@@ -68,15 +68,15 @@
     <inertial>
       <origin
-        xyz="5.24591222383746E-06 -0.00359346563883705 0.138355957541882"
-        rpy="0 0 0" />
-      <mass
-        value="9.69438463218994" />
-      <inertia
-        ixx="0.087356099909061"
-        ixy="7.53498644731024E-06"
-        ixz="-1.01700173972257E-05"
-        iyy="0.0784434736574001"
-        iyz="0.00201488298749374"
-        izz="0.058685623931688" />
+        xyz="8.07683021386315E-06 -0.0035773925820559 0.146117252792634"
+        rpy="0 0 0" />
+      <mass
+        value="9.69439879854905" />
+      <inertia
+        ixx="0.0873560745698383"
+        ixy="7.48773843082023E-06"
+        ixz="-1.01202228048275E-05"
+        iyy="0.0784436265757321"
+        iyz="0.0020149616199151"
+        izz="0.0586857551015982" />
     </inertial>
     <visual>
@@ -108,8 +108,8 @@
     type="revolute">
     <origin
-      xyz="0 1.592E-05 0.087761"
-      rpy="0 0 0" />
-    <parent
-      link="elfin_base" />
+      xyz="0 0 0.08"
+      rpy="0 0 0" />
+    <parent
+      link="base_link" />
     <child
       link="elfin_link1" />
@@ -126,15 +126,15 @@
     <inertial>
       <origin
-        xyz="1.95251384530923E-05 -0.0416913324558573 0.292090528307612"
-        rpy="0 0 0" />
-      <mass
-        value="9.54888007421455" />
-      <inertia
-        ixx="0.589316020458646"
-        ixy="4.87072038508207E-06"
-        ixz="-5.64092391701446E-05"
-        iyy="0.596073639080168"
-        iyz="-0.0314560812525604"
-        izz="0.0224324476203139" />
+        xyz="2.00668503935044E-05 -0.0350913888576602 0.29208552291378"
+        rpy="0 0 0" />
+      <mass
+        value="9.54892004428153" />
+      <inertia
+        ixx="0.589306179672266"
+        ixy="4.62108054755441E-06"
+        ixz="-5.92121709739712E-05"
+        iyy="0.59606406844587"
+        iyz="-0.0314540755137635"
+        izz="0.0224322625270061" />
     </inertial>
     <visual>
@@ -166,5 +166,5 @@
     type="revolute">
     <origin
-      xyz="0 -0.11237 0.17424"
+      xyz="0 -0.11895 0.182"
       rpy="0 0 0" />
     <parent
@@ -184,15 +184,15 @@
     <inertial>
       <origin
-        xyz="-2.05498098492835E-07 0.0805813619575155 0.0369739757853127"
-        rpy="0 0 0" />
-      <mass
-        value="2.91695075996986" />
-      <inertia
-        ixx="0.0135717990039811"
-        ixy="-2.96883650370101E-07"
-        ixz="4.86606934151349E-07"
-        iyy="0.0118099746880734"
-        iyz="-0.000536934244185151"
-        izz="0.00742981276706272" />
+        xyz="-3.35410138302954E-06 0.0807007389842829 0.0361017927579714"
+        rpy="0 0 0" />
+      <mass
+        value="2.9169641646369" />
+      <inertia
+        ixx="0.0135718271521769"
+        ixy="-2.93064412428029E-07"
+        ixz="4.8594264368378E-07"
+        iyy="0.0118099812788293"
+        iyz="-0.000536922283164078"
+        izz="0.00742983650345206" />
     </inertial>
     <visual>
@@ -224,5 +224,5 @@
     type="revolute">
     <origin
-      xyz="0 0.0274 0.72913"
+      xyz="0 0.03388 0.73"
       rpy="0 0 0" />
     <parent
@@ -242,15 +242,15 @@
     <inertial>
       <origin
-        xyz="3.96873522626768E-05 -0.0650155011553575 0.173832874640951"
-        rpy="0 0 0" />
-      <mass
-        value="2.82013622855012" />
-      <inertia
-        ixx="0.0599767754983424"
-        ixy="3.79711278884469E-06"
-        ixz="-1.98444520902161E-05"
-        iyy="0.0558250057132048"
-        iyz="0.0126917031165999"
-        izz="0.00791935397298624" />
+        xyz="3.96870930380675E-05 -0.0650155014813431 0.173832877361676"
+        rpy="0 0 0" />
+      <mass
+        value="2.82013626298568" />
+      <inertia
+        ixx="0.0599767847611795"
+        ixy="3.79703423156232E-06"
+        ixz="-1.98457784458686E-05"
+        iyy="0.0558250152691264"
+        iyz="0.0126917028887549"
+        izz="0.00791935431280652" />
     </inertial>
     <visual>
@@ -265,5 +265,5 @@
         name="">
         <color
-          rgba="0.792156862745098 0.819607843137255 0.933333333333333 1" />
+          rgba="1 1 1 1" />
       </material>
     </visual>
@@ -282,5 +282,5 @@
     type="revolute">
     <origin
-      xyz="0 0.08495 0.14787"
+      xyz="0 0.08507 0.147"
       rpy="0 0 0" />
     <parent
@@ -300,15 +300,15 @@
     <inertial>
       <origin
-        xyz="0.000106591955597646 0.0685097048909167 0.0256514039444942"
-        rpy="0 0 0" />
-      <mass
-        value="1.25663090248721" />
-      <inertia
-        ixx="0.00349957647668621"
-        ixy="-4.75533746465021E-07"
-        ixz="-2.50320892962122E-07"
-        iyy="0.00273058830542026"
-        iyz="-9.97554673070372E-05"
-        izz="0.00202568589371655" />
+        xyz="7.12907192415623E-06 0.0685097120449843 0.0250239802320473"
+        rpy="0 0 0" />
+      <mass
+        value="1.25663358547766" />
+      <inertia
+        ixx="0.00349953854194773"
+        ixy="-4.77573905026001E-07"
+        ixz="-2.77272767775186E-07"
+        iyy="0.00273055902205603"
+        iyz="-9.97691077673872E-05"
+        izz="0.00202572610862977" />
     </inertial>
     <visual>
@@ -340,5 +340,5 @@
     type="revolute">
     <origin
-      xyz="-9.9457E-05 -0.071 0.42237"
+      xyz="0 -0.071 0.423"
       rpy="0 0 0" />
     <parent
@@ -358,15 +358,15 @@
     <inertial>
       <origin
-        xyz="0.000340707255698251 -8.81908601502805E-05 0.029796591504043"
-        rpy="0 0 0" />
-      <mass
-        value="0.347759299047143" />
-      <inertia
-        ixx="0.000251824751508589"
-        ixy="3.78375395442371E-08"
-        ixz="2.36891401002385E-07"
-        iyy="0.00025253810450235"
-        iyz="-2.61455738317234E-08"
-        izz="0.000309218893868899" />
+        xyz="0.000340707984155859 -8.81908556493069E-05 0.0297965916937253"
+        rpy="0 0 0" />
+      <mass
+        value="0.347759307077889" />
+      <inertia
+        ixx="0.000251824752714629"
+        ixy="3.78375113977756E-08"
+        ixz="2.3688911249132E-07"
+        iyy="0.000252538114035222"
+        iyz="-2.61458838436258E-08"
+        izz="0.000309218903006093" />
     </inertial>
     <visual>
@@ -398,5 +398,5 @@
     type="revolute">
     <origin
-      xyz="9.9456E-05 0.071 0.11163"
+      xyz="0 0.071 0.111"
       rpy="0 0 0" />
     <parent
@@ -417,5 +417,5 @@
     type="fixed">
     <origin
-      xyz="0 0 0.0599"
+      xyz="0 0 0.0625"
       rpy="0 0 0" />
     <parent
